File: Spear_hw/Spear.kicad_pcb (KiCad board)
At the start: 4 copper layers, 18 x 84 mm, 83 parts, among them Q1 2N7002, Q2 IRF9317, Q3 IRLML6401, Q4 2N7002, SW1 BUTTON, SW2 BUTTON

Commit message: + RadioSpear HW
Parts:
- removed C1: 10n, Capacitors:CAP_0603_Silks
- removed XL10: CONN_2, PCB:Oval3x1.5wHole0d9_x2
- removed XL9: CONN_3, Connectors:SLD_3_2D5
- added R8: 10k, Resistors:RES_0603, B.Cu at (141.2, 122.5)
- added TP3: TESTPOINT, PCB:TESTPOINT_1MM, F.Cu at (138.9, 136.8)
- ANT1: footprint Antennas:MagicStick -> Antennas:ANT_868_Spear_inverted
- DA4: value ST1CC40_SO8 -> ST1CC40
- R1: value 1M -> 1k; moved to B.Cu
- XL5: value CONN_2 -> CONN_3; footprint Connectors:WB-02(MW-2M) -> Connectors:WB-03(MW-3M)
- moved XL4 48.5 mm to (140.2, 59.1)
- moved R1 13.7 mm to (139.7, 148.6), turned to 180 degrees
- moved Logo1 13.5 mm to (145.4, 96.7), turned to 0 degrees
- moved R2 4.03 mm to (144.9, 118.5), turned to 90 degrees
- moved C5 3.42 mm to (139.2, 106.8)
- moved DA1 3.41 mm to (139.1, 109.3)
- moved Q2 3.34 mm to (139.9, 109.6)
- moved R3 3.15 mm to (138.9, 112.2)
- moved XL2 3.14 mm to (138.8, 115.9)
- moved ANT1 1.59 mm to (145.4, 105.0), turned to 0 degrees
- moved XL5 1.30 mm to (138.8, 123.6)
- moved XL6 0.32 mm to (138.8, 130.9)
- moved Q1 0.14 mm to (142.1, 118.5), turned to 90 degrees
- turned SW1 to 0 degrees
- turned TP1 to 180 degrees
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Connections:
- net Net-(DD1-Pad11) renamed /BTN2
- DD1 pad 13: (no net) -> Net-(DD1-Pad13)
- DD1 pad 14: (no net) -> /NPX_PWR_EN
- DD1 pad 15: (no net) -> Net-(DD1-Pad15)
- DD1 pad 16: /NPX_PWR_EN -> Net-(DD1-Pad15)
- R1 pad 1: Net-(C1-Pad2) -> Net-(DD1-Pad13)
- R1 pad 2: GND -> /5V_USB
- XL3 pad H1: Net-(C1-Pad2) -> Net-(XL3-PadH1)
- XL3 pad H2: Net-(C1-Pad2) -> (no net)
- XL3 pad H3: Net-(C1-Pad2) -> (no net)
- XL3 pad H4: Net-(C1-Pad2) -> Net-(XL3-PadH4)
- XL5 pad 1: /BTN1 -> GND
- XL5 pad 2: +3v3 -> /BTN1
Routing:
- net Net-(DA4-Pad5): track 83.3 -> 18.1 mm
- net Net-(C37-Pad1): track 69.9 -> 4.79 mm
- net GND: track 253.8 -> 286.1 mm, vias 45 -> 50
- net Net-(C1-Pad2): track 17.2 -> 0.00 mm
- net Net-(DD1-Pad13): track 0.00 -> 13.7 mm, vias 0 -> 2
- net /NPX_PWR: track 47.0 -> 59.0 mm, vias 0 -> 1
- net /DIN0: track 44.7 -> 54.1 mm, vias 1 -> 0
- net Net-(DD1-Pad15): track 0.00 -> 6.41 mm
- net /BTN1: track 31.2 -> 37.0 mm
- net /5V_USB: track 31.7 -> 36.6 mm
- net /NPX1_CTRL: track 30.1 -> 34.6 mm
- net Net-(Q1-Pad3): track 4.64 -> 8.67 mm
- net /NPX_PWR_EN: track 22.3 -> 26.0 mm
- net Net-(XL3-PadH4): track 0.00 -> 3.16 mm
- net Net-(XL3-PadH1): track 0.00 -> 3.16 mm
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- removed copper zone on In1.Cu, net /NPX_PWR
- removed copper zone on In2.Cu, net /NPX_PWR
Other:
- board size 18 x 84 mm -> 18 x 96 mm
- net class Default: via_dia 0.65 -> 0.6
- net class Wide: via_dia 0.65 -> 0.6
- rule via_min_size: 0.4 -> 0.6
- board text added: "+"
- board text added: "-"
- board text added: "Charger"
- board text added: "Data"
- board text added: "Ostranna RadioSpear v1.0"
- board text added: "ST1CC40"
