File: Spear_hw/Spear.sch (KiCad schematic (older format))
At the start: 83 parts, among them Q1 2N7002, Q2 IRF9317, Q3 IRLML6401, Q4 2N7002, SW1 BUTTON, SW2 BUTTON

Commit message: + RadioSpear HW
Parts:
- removed C1: 10n, Capacitors:CAP_0603_Silks, symbol Tittar_kl:C
- removed XL10: CONN_2, PCB:Oval3x1.5wHole0d9_x2, symbol Connectors_kl:CONN_2
- removed XL5: CONN_2, Connectors:WB-02(MW-2M), symbol Connectors_kl:CONN_2
- removed XL9: CONN_3, Connectors:SLD_3_2D5, symbol Connectors_kl:CONN_3
- added R8: 10k, Resistors:RES_0603, symbol Tittar_kl:R
- added TP3: TESTPOINT, PCB:TESTPOINT_1MM, symbol pcb_details:TESTPOINT
- added XL5: CONN_3, Connectors:WB-03(MW-3M), symbol Connectors_kl:CONN_3
- ANT1: footprint Antennas:MagicStick -> Antennas:ANT_868_Spear_inverted
- R1: value 1M -> 1k
Connections:
- net +3v3: now also XL5.3
- net 5V_USB: now also R1.2
- net BTN1: now also R8.1, XL5.2 (PM)
- net GND: now also R8.2, XL5.1 (P1); no longer R1.2
- net NPX_PWR_EN: now also DD1.14 (ADC9/SAI1FSB/LPTIM2_OUT/DAC1/CK2/PA4); no longer DD1.16 (ADC11/T16C1/MISO1/PA6)
- net BTN2: now reaches DD1.11 (ADC6/T2C2/T15C1N/SCK1/PA1), SW2.1, XL6.1 (P1)
- net at DD1.13 (ADC8/SAI1MCLKA/T15C2/T2C4/LP1RX/RX2/PA3): now also R1.1
- net at DD1.15 (ADC10/T2C1ETR/DAC2/SCK1/PA5): now also DD1.16 (ADC11/T16C1/MISO1/PA6), TP3.1
- now unconnected: XL3.H1, XL3.H2, XL3.H3, XL3.H4
- no-connect marks 13 -> 14
Other:
- note added: "LED driver"
- note added: "NPX clock"
- note removed: "LED drivers"
- moved on the sheet: C10, C11, C12, C13, C14, C15, C16, C17, C18, C19, C2, C20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
